File: AtkDongle.kicad_pcb (KiCad board)
At the start: 2 copper layers, 30.3 x 35.8 mm, 12 parts, among them J1 PARALLEL_SIDE, J2 SERIAL_SIDE, J99 OSHW_LOGO, P1 +5V, P2 +12V, P3 -12V

Commit message: Ready for prototypes!
Parts:
- added TP1: TP+5V, TestPoint:TestPoint_Pad_D2.0mm, F.Cu at (116.8, 119.1)
- added TP2: TP+12V, TestPoint:TestPoint_Pad_D2.0mm, F.Cu at (112.4, 119.1)
- added TP3: TP-12V, TestPoint:TestPoint_Pad_D2.0mm, F.Cu at (121.3, 119.1)
- added TP4: TPGND, TestPoint:TestPoint_Pad_D2.0mm, F.Cu at (116.8, 88.8)
- moved J99 0.05 mm to (116.8, 117.9)
Routing:
- net -12V: track 22.1 -> 46.3 mm, vias 0 -> 1
- net +12V: track 21.2 -> 36.4 mm
- net +5V: track 18.3 -> 25.1 mm
- net GND: vias 0 -> 19
Other:
- board text added: "V1"
Changed lines of the file:
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@@
   (general
     (thickness 1.6)
-    (drawings 15)
-    (tracks 65)
+    (drawings 20)
+    (tracks 93)
     (zones 0)
-    (modules 12)
+    (modules 16)
     (nets 17)
   )
   (page A4)
+  (title_block
+    (title AtkDonge)
+    (date 2020-01-02)
+    (rev 1git)
+    (company SukkoPera)
+  )
   (layers
     (0 F.Cu signal)
@@
     (mod_text_size 1 1)
     (mod_text_width 0.15)
-    (pad_size 1.8 1.8)
-    (pad_drill 0.9)
+    (pad_size 2 2)
+    (pad_drill 0)
     (pad_to_mask_clearance 0)
     (solder_mask_min_width 0.25)
@@
     (visible_elements FFFFFF7F)
     (pcbplotparams
-      (layerselection 0x010fc_ffffffff)
+      (layerselection 0x010f0_ffffffff)
       (usegerberextensions false)
       (usegerberattributes false)
@@
       (outputformat 1)
       (mirror false)
-      (drillshape 1)
+      (drillshape 0)
       (scaleselection 1)
-      (outputdirectory ""))
+      (outputdirectory "gerbers"))
   )
   (net 0 "")
@@
   )
   (module Symbol:OSHW-Logo2_7.3x6mm_Copper (layer B.Cu)
-    (at 116.7892 117.856 180)
+    (at 116.84 117.856 180)
     (descr "Open Source Hardware Symbol")
     (tags "Logo Symbol OSHW")
@@
       (xy -0.113933 2.757629) (xy -0.013056 2.757714) (xy 0 2.757714) (xy 0.10391 2.757652)) (layer B.Cu) (width 0.01))
   )
+  (module TestPoint:TestPoint_Pad_D2.0mm (layer F.Cu)
+    (at 116.84 119.126)
+    (descr "SMD pad as test Point, diameter 2.0mm")
+    (tags "test point SMD pad")
+    (attr virtual)
+    (fp_text reference TP1 (at 0 -1.998) (layer F.SilkS) hide
+      (effects (font (size 1 1) (thickness 0.15)))
+    )
+    (fp_text value TP+5V (at 0 2.05) (layer F.Fab)
+      (effects (font (size 1 1) (thickness 0.15)))
+    )
+    (fp_text user %R (at 0 -2) (layer F.Fab)
+      (effects (font (size 1 1) (thickness 0.15)))
+    )
+    (fp_circle (center 0 0) (end 1.5 0) (layer F.CrtYd) (width 0.05))
+    (fp_circle (center 0 0) (end 0 1.2) (layer F.SilkS) (width 0.12))
+    (pad 1 smd circle (at 0 0) (size 2 2) (layers F.Cu F.Mask)
+      (net 13 +5V))
+  )
+  (module TestPoint:TestPoint_Pad_D2.0mm (layer F.Cu)
+    (at 112.395 119.126)
+    (descr "SMD pad as test Point, diameter 2.0mm")
+    (tags "test point SMD pad")
+    (attr virtual)
+    (fp_text reference TP2 (at 0 -1.998) (layer F.SilkS) hide
+      (effects (font (size 1 1) (thickness 0.15)))
+    )
+    (fp_text value TP+12V (at 0 2.05) (layer F.Fab)
+      (effects (font (size 1 1) (thickness 0.15)))
+    )
+    (fp_circle (center 0 0) (end 0 1.2) (layer F.SilkS) (width 0.12))
+    (fp_circle (center 0 0) (end 1.5 0) (layer F.CrtYd) (width 0.05))
+    (fp_text user %R (at 0 -2) (layer F.Fab)
+      (effects (font (size 1 1) (thickness 0.15)))
+    )
+    (pad 1 smd circle (at 0 0) (size 2 2) (layers F.Cu F.Mask)
+      (net 14 +12V))
+  )
+  (module TestPoint:TestPoint_Pad_D2.0mm (layer F.Cu)
+    (at 121.285 119.126)
+    (descr "SMD pad as test Point, diameter 2.0mm")
+    (tags "test point SMD pad")
+    (attr virtual)
+    (fp_text reference TP3 (at 0 -1.998) (layer F.SilkS) hide
+      (effects (font (size 1 1) (thickness 0.15)))
+    )
+    (fp_text value TP-12V (at 0 2.05) (layer F.Fab)
+      (effects (font (size 1 1) (thickness 0.15)))
+    )
+    (fp_text user %R (at 0 -2) (layer F.Fab)
+      (effects (font (size 1 1) (thickness 0.15)))
+    )
+    (fp_circle (center 0 0) (end 1.5 0) (layer F.CrtYd) (width 0.05))
+    (fp_circle (center 0 0) (end 0 1.2) (layer F.SilkS) (width 0.12))
+    (pad 1 smd circle (at 0 0) (size 2 2) (layers F.Cu F.Mask)
+      (net 15 -12V))
+  )
+  (module TestPoint:TestPoint_Pad_D2.0mm (layer F.Cu)
+    (at 116.84 88.778)
+    (descr "SMD pad as test Point, diameter 2.0mm")
+    (tags "test point SMD pad")
+    (attr virtual)
+    (fp_text reference TP4 (at 0 -1.998) (layer F.SilkS) hide
+      (effects (font (size 1 1) (thickness 0.15)))
+    )
+    (fp_text value TPGND (at 0 2.05) (layer F.Fab)
+      (effects (font (size 1 1) (thickness 0.15)))
+    )
+    (fp_circle (center 0 0) (end 0 1.2) (layer F.SilkS) (width 0.12))
+    (fp_circle (center 0 0) (end 1.5 0) (layer F.CrtYd) (width 0.05))
+    (fp_text user %R (at 0 -2) (layer F.Fab)
+      (effects (font (size 1 1) (thickness 0.15)))
+    )
+    (pad 1 smd circle (at 0 0) (size 2 2) (layers F.Cu F.Mask)
+      (net 16 GND))
+  )
+  (gr_text V1 (at 107.188 121.031) (layer B.SilkS)
+    (effects (font (size 1 1) (thickness 0.15)) (justify mirror))
+  )
+  (gr_text -12V (at 121.285 121.285) (layer F.SilkS)
+    (effects (font (size 1 1) (thickness 0.15)))
+  )
+  (gr_text +12V (at 112.395 121.285) (layer F.SilkS)
+    (effects (font (size 1 1) (thickness 0.15)))
+  )
+  (gr_text +5V (at 116.84 121.285) (layer F.SilkS)
+    (effects (font (size 1 1) (thickness 0.15)))
+  )
+  (gr_text GND (at 119.888 88.7105) (layer F.SilkS)
+    (effects (font (size 1 1) (thickness 0.15)))
+  )
   (gr_text "Licensed\nunder CERN\nOHL v.1.2" (at 116.7892 108.6085) (layer B.SilkS)
     (effects (font (size 1 1) (thickness 0.15)) (justify mirror))
@@
     (effects (font (size 1 1) (thickness 0.15)))
   )
-  (gr_text GND (at 124.9303 116.332 90) (layer F.SilkS)
+  (gr_text GND (at 124.9303 115.951 90) (layer F.SilkS)
     (effects (font (size 1 1) (thickness 0.15)))
   )
-  (gr_text +5V (at 122.3903 116.332 90) (layer F.SilkS)
+  (gr_text +5V (at 122.3903 115.951 90) (layer F.SilkS)
     (effects (font (size 1 1) (thickness 0.15)))
   )
@@
   (segment (start 122.4578 112.831) (end 122.4578 118.9018) (width 0.5) (layer B.Cu) (net 13) (status 10))
   (segment (start 123.312 119.756) (end 129.9464 119.756) (width 0.5) (layer B.Cu) (net 13) (status 20))
+  (segment (start 118.0542 117.9118) (end 116.84 119.126) (width 0.5) (layer F.Cu) (net 13))
+  (segment (start 118.0542 112.831) (end 118.0542 117.9118) (width 0.5) (layer F.Cu) (net 13))
   (segment (start 103.632 98.981) (end 114.475 98.981) (width 0.5) (layer F.Cu) (net 14) (status 10))
   (segment (start 115.5242 100.0302) (end 115.5242 104.521) (width 0.5) (layer F.Cu) (net 14) (status 20))
   (segment (start 114.475 98.981) (end 115.5242 100.0302) (width 0.5) (layer F.Cu) (net 14))
   (segment (start 115.5242 104.521) (end 111.120599 104.521) (width 0.5) (layer F.Cu) (net 14) (status 30))
+  (segment (start 112.395 105.795401) (end 111.120599 104.521) (width 0.5) (layer F.Cu) (net 14))
+  (segment (start 112.395 119.126) (end 112.395 105.795401) (width 0.5) (layer F.Cu) (net 14))
   (segment (start 115.5142 96.211) (end 103.632 96.211) (width 0.5) (layer F.Cu) (net 15) (status 30))
   (segment (start 115.5142 95.0518) (end 115.5142 96.211) (width 0.5) (layer B.Cu) (net 15) (status 20))
@@
   (segment (start 122.4578 95.008919) (end 121.428881 93.98) (width 0.5) (layer B.Cu) (net 15))
   (segment (start 122.4578 96.211) (end 122.4578 95.008919) (width 0.5) (layer B.Cu) (net 15) (status 10))
+  (via (at 120.285001 105.664) (size 0.8) (drill 0.6) (layers F.Cu B.Cu) (net 15))
+  (segment (start 121.285 119.126) (end 120.285001 118.126001) (width 0.5) (layer F.Cu) (net 15))
+  (segment (start 120.285001 118.126001) (end 120.285001 105.680001) (width 0.5) (layer F.Cu) (net 15))
+  (segment (start 120.285001 98.383799) (end 122.4578 96.211) (width 0.5) (layer B.Cu) (net 15))
+  (segment (start 120.285001 105.664) (end 120.285001 98.383799) (width 0.5) (layer B.Cu) (net 15))
   (segment (start 103.632 104.521) (end 108.580599 104.521) (width 0.5) (layer F.Cu) (net 16) (status 30))
   (segment (start 124.9978 112.831) (end 124.9978 110.4094) (width 0.5) (layer B.Cu) (net 16) (status 10))
   (segment (start 126.7312 108.676) (end 129.9464 108.676) (width 0.5) (layer B.Cu) (net 16) (status 20))
   (segment (start 124.9978 110.4094) (end 126.7312 108.676) (width 0.5) (layer B.Cu) (net 16))
+  (via (at 122.4578 103.251) (size 0.8) (drill 0.6) (layers F.Cu B.Cu) (net 16))
+  (via (at 124.9978 103.251) (size 0.8) (drill 0.6) (layers F.Cu B.Cu) (net 16))
+  (via (at 124.9978 92.473) (size 0.8) (drill 0.6) (layers F.Cu B.Cu) (net 16))
+  (via (at 122.4578 92.473) (size 0.8) (drill 0.6) (layers F.Cu B.Cu) (net 16))
+  (via (at 111.120599 87.901) (size 0.8) (drill 0.6) (layers F.Cu B.Cu) (net 16))
+  (via (at 108.580599 87.901) (size 0.8) (drill 0.6) (layers F.Cu B.Cu) (net 16))
+  (via (at 124.9978 87.901) (size 0.8) (drill 0.6) (layers F.Cu B.Cu) (net 16))
+  (via (at 122.4578 87.901) (size 0.8) (drill 0.6) (layers F.Cu B.Cu) (net 16))
+  (via (at 111.120599 92.473) (size 0.8) (drill 0.6) (layers F.Cu B.Cu) (net 16))
+  (via (at 108.580599 92.473) (size 0.8) (drill 0.6) (layers F.Cu B.Cu) (net 16))
+  (via (at 111.120599 97.68) (size 0.8) (drill 0.6) (layers F.Cu B.Cu) (net 16))
+  (via (at 108.580599 97.68) (size 0.8) (drill 0.6) (layers F.Cu B.Cu) (net 16))
+  (via (at 118.0542 101.604401) (size 0.8) (drill 0.6) (layers F.Cu B.Cu) (net 16))
+  (via (at 118.0542 99.064401) (size 0.8) (drill 0.6) (layers F.Cu B.Cu) (net 16))
+  (via (at 118.745 121.158) (size 0.8) (drill 0.6) (layers F.Cu B.Cu) (net 16))
+  (via (at 114.808 121.175) (size 0.8) (drill 0.6) (layers F.Cu B.Cu) (net 16))
+  (via (at 124.9978 121.175) (size 0.8) (drill 0.6) (layers F.Cu B.Cu) (net 16))
+  (via (at 108.580599 121.175) (size 0.8) (drill 0.6) (layers F.Cu B.Cu) (net 16))
+  (via (at 116.7842 108.843401) (size 0.8) (drill 0.6) (layers F.Cu B.Cu) (net 16))
   (zone (net 16) (net_name GND) (layer F.Cu) (hatch edge 0.508)
     (connect_pads (clearance 0.254))
